Commit message: Actualización adicional - AGENTS.md y documentación

File: install/cr20_moveit/share/cr20_moveit/config/cr20_robot.ros2_control.xacro (robot description, xacro)
@@ -1,54 +1 @@
-<?xml version="1.0"?>
-<robot xmlns:xacro="http://www.ros.org/wiki/xacro">
-    <xacro:macro name="cr20_robot_ros2_control" params="name initial_positions_file">
-        <xacro:property name="initial_positions" value="${load_yaml(initial_positions_file)['initial_positions']}"/>
-        <ros2_control name="${name}" type="system">
-            <hardware>
-                <!-- By default, set up controllers for simulation. This won't work on real hardware -->
-                <plugin>mock_components/GenericSystem</plugin>
-            </hardware>
-            <joint name="joint1">
-                <command_interface name="position"/>
-                <state_interface name="position">
-                  <param name="initial_value">${initial_positions['joint1']}</param>
-                </state_interface>
-                <state_interface name="velocity"/>
-            </joint>
-            <joint name="joint2">
-                <command_interface name="position"/>
-                <state_interface name="position">
-                  <param name="initial_value">${initial_positions['joint2']}</param>
-                </state_interface>
-                <state_interface name="velocity"/>
-            </joint>
-            <joint name="joint3">
-                <command_interface name="position"/>
-                <state_interface name="position">
-                  <param name="initial_value">${initial_positions['joint3']}</param>
-                </state_interface>
-                <state_interface name="velocity"/>
-            </joint>
-            <joint name="joint4">
-                <command_interface name="position"/>
-                <state_interface name="position">
-                  <param name="initial_value">${initial_positions['joint4']}</param>
-                </state_interface>
-                <state_interface name="velocity"/>
-            </joint>
-            <joint name="joint5">
-                <command_interface name="position"/>
-                <state_interface name="position">
-                  <param name="initial_value">${initial_positions['joint5']}</param>
-                </state_interface>
-                <state_interface name="velocity"/>
-            </joint>
-            <joint name="joint6">
-                <command_interface name="position"/>
-                <state_interface name="position">
-                  <param name="initial_value">${initial_positions['joint6']}</param>
-                </state_interface>
-                <state_interface name="velocity"/>
-            </joint>
-        </ros2_control>
-    </xacro:macro>
-</robot>
+/home/iudc/dobot_ws/src/DOBOT_6Axis_ROS2_V4/cr20_moveit/config/cr20_robot.ros2_control.xacro

File: install/cr20_moveit/share/cr20_moveit/config/cr20_robot.urdf.xacro (robot description, xacro)
@@ -1,9 +1 @@
-<?xml version="1.0"?>
-<robot xmlns:xacro="http://www.ros.org/wiki/xacro" name="cr20_robot">
-    <xacro:arg name="initial_positions_file" default="initial_positions.yaml" />
-    <!-- Import cr20_robot urdf file -->
-    <xacro:include filename="$(find dobot_rviz)/urdf/cr20_robot.urdf" />
-    <!-- Import control_xacro -->
-    <xacro:include filename="cr20_robot.ros2_control.xacro" />
-    <xacro:cr20_robot_ros2_control name="FakeSystem" initial_positions_file="$(arg initial_positions_file)"/>
-</robot>
+/home/iudc/dobot_ws/src/DOBOT_6Axis_ROS2_V4/cr20_moveit/config/cr20_robot.urdf.xacro

File: install/cra_description/share/cra_description/urdf/camera_ceiling.urdf.xacro (robot description, xacro)
@@ -1,11 +1 @@
-<?xml version="1.0"?>
-<robot xmlns:xacro="http://www.ros.org/wiki/xacro" name="ceiling_camera">
-  <!-- Include our wrapper that extends official model -->
-  <xacro:include filename="$(find cra_description)/urdf/d435i_with_gazebo.urdf.xacro"/>
-  <!-- World link -->
-  <link name="world"/>
-  <!-- Mount camera in ceiling using extended model -->
-  <xacro:d435i_with_gazebo parent="world" name="camera" use_nominal_extrinsics="true">
-    <origin xyz="0 0 3.0" rpy="0 ${pi/2} 0"/>
-  </xacro:d435i_with_gazebo>
-</robot>
+/home/iudc/dobot_ws/src/DOBOT_6Axis_ROS2_V4/cra_description/urdf/camera_ceiling.urdf.xacro

File: install/cra_description/share/cra_description/urdf/camera_setup.urdf.xacro (robot description, xacro)
@@ -1,31 +1 @@
-<?xml version="1.0"?>
-<robot xmlns:xacro="http://www.ros.org/wiki/xacro" name="camera_setup">
-  <!-- Include RealSense D435i -->
-  <xacro:include filename="$(find realsense2_description)/urdf/_d435i.urdf.xacro"/>
-  <!-- World link (reference point) -->
-  <link name="world"/>
-  <!-- Camera mount link (ceiling) -->
-  <link name="camera_mount">
-    <visual>
-      <origin xyz="0 0 -0.05" rpy="0 0 0"/>
-      <geometry>
-        <cylinder radius="0.05" length="0.1"/>
-      </geometry>
-      <material name="mount_grey">
-        <color rgba="0.5 0.5 0.5 1.0"/>
-      </material>
-    </visual>
-  </link>
-  <!-- Mount camera to world (ceiling position) -->
-  <joint name="camera_mount_joint" type="fixed">
-    <parent link="world"/>
-    <child link="camera_mount"/>
-    <!-- Position: X=0, Y=0, Z=2.0 metros (altura del techo) -->
-    <origin xyz="0 0 2.0" rpy="0 0 0"/>
-  </joint>
-  <!-- Attach D435i camera pointing down -->
-  <xacro:sensor_d435i parent="camera_mount" name="camera" use_nominal_extrinsics="true">
-    <!-- Rotate -90 degrees in pitch to point downward -->
-    <origin xyz="0 0 0" rpy="0 ${pi/2} 0"/>
-  </xacro:sensor_d435i>
-</robot>
+/home/iudc/dobot_ws/src/DOBOT_6Axis_ROS2_V4/cra_description/urdf/camera_setup.urdf.xacro

File: install/cra_description/share/cra_description/urdf/cr20_robot.xacro (robot description, xacro)
@@ -1,474 +1 @@
-<?xml version="1.0" encoding="utf-8"?>
-<robot
-  name="cr20_robot" xmlns:xacro="http://ros.org/wiki/xacro">
-  <link name="dummy_link"/>
-  <link
-    name="base_link">
-    <inertial>
-      <origin
-        xyz="-0.0523349568972135 0.0899270486094572 -0.00279275668479641"
-        rpy="0 0 0" />
-      <mass
-        value="5.0" />
-      <inertia
-        ixx="0.01"
-        ixy="0"
-        ixz="0"
-        iyy="0.01"
-        iyz="0"
-        izz="0.01" />
-    </inertial>
-    <visual>
-      <origin
-        xyz="0 0 0"
-        rpy="0 0 0" />
-      <geometry>
-        <mesh
-          filename="file://$(find cra_description)/meshes/cr20/base_link.STL" />
-      </geometry>
-      <material
-        name="">
-        <color
-          rgba="0.792156862745098 0.819607843137255 0.933333333333333 1" />
-      </material>
-    </visual>
-    <collision>
-      <origin
-        xyz="0 0 0"
-        rpy="0 0 0" />
-      <geometry>
-        <mesh
-          filename="file://$(find cra_description)/meshes/cr20/base_link.STL" />
-      </geometry>
-    </collision>
-  </link>
-  <link name="world"/>
-  <joint name="world_joint" type="fixed">
-    <origin xyz="0 0 0.03" rpy="0 0 0" />
-    <parent link="world" />
-    <child  link="dummy_link" />
-  </joint>
-  <joint name="dummy_joint" type="fixed">
-    <parent link="dummy_link" />
-    <child  link="base_link" />
-  </joint>
-  <link
-    name="Link1">
-    <inertial>
-      <origin
-        xyz="-0.0154576425326206 -0.0986375365415087 1.04119647925812"
-        rpy="0 0 0" />
-      <mass
-        value="8.0" />
-      <inertia
-        ixx="0.05"
-        ixy="0"
-        ixz="0"
-        iyy="0.05"
-        iyz="0"
-        izz="0.02" />
-    </inertial>
-    <visual>
-      <origin
-        xyz="0 0 0"
-        rpy="0 0 0" />
-      <geometry>
-        <mesh
-          filename="file://$(find cra_description)/meshes/cr20/Link1.STL" />
-      </geometry>
-      <material
-        name="">
-        <color
-          rgba="0.792156862745098 0.819607843137255 0.933333333333333 1" />
-      </material>
-    </visual>
-    <collision>
-      <origin
-        xyz="0 0 0"
-        rpy="0 0 0" />
-      <geometry>
-        <mesh
-          filename="file://$(find cra_description)/meshes/cr20/Link1.STL" />
-      </geometry>
-    </collision>
-  </link>
-  <joint
-    name="joint1"
-    type="revolute">
-    <origin
-      xyz="0 0 0.23"
-      rpy="0 0 0" />
-    <parent
-      link="base_link" />
-    <child
-      link="Link1" />
-    <axis
-      xyz="0 0 1" />
-    <limit
-      lower="-6.28"
-      upper="6.28"
-      effort="150"
-      velocity="3.14" />
-  </joint>
-  <link
-    name="Link2">
-    <inertial>
-      <origin
-        xyz="-0.828898669983325 -3.97165169431493E-07 0.115283168336158"
-        rpy="0 0 0" />
-      <mass
-        value="6.0" />
-      <inertia
-        ixx="0.1"
-        ixy="0"
-        ixz="0"
-        iyy="0.1"
-        iyz="0"
-        izz="0.02" />
-    </inertial>
-    <visual>
-      <origin
-        xyz="0 0 0"
-        rpy="0 0 0" />
-      <geometry>
-        <mesh
-          filename="file://$(find cra_description)/meshes/cr20/Link2.STL" />
-      </geometry>
-      <material
-        name="">
-        <color
-          rgba="0.792156862745098 0.819607843137255 0.933333333333333 1" />
-      </material>
-    </visual>
-    <collision>
-      <origin
-        xyz="0 0 0"
-        rpy="0 0 0" />
-      <geometry>
-        <mesh
-          filename="file://$(find cra_description)/meshes/cr20/Link2.STL" />
-      </geometry>
-    </collision>
-  </link>
-  <joint
-    name="joint2"
-    type="revolute">
-    <origin
-      xyz="0 0 0"
-      rpy="1.5708 1.5708 0" />
-    <parent
-      link="Link1" />
-    <child
-      link="Link2" />
-    <axis
-      xyz="0 0 1" />
-    <limit
-      lower="-6.28"
-      upper="6.28"
-      effort="150"
-      velocity="3.14" />
-  </joint>
-  <link
-    name="Link3">
-    <inertial>
-      <origin
-        xyz="-0.746000007821945 1.07337005127015E-07 0.0757301295800403"
-        rpy="0 0 0" />
-      <mass
-        value="4.0" />
-      <inertia
-        ixx="0.05"
-        ixy="0"
-        ixz="0"
-        iyy="0.05"
-        iyz="0"
-        izz="0.01" />
-    </inertial>
-    <visual>
-      <origin
-        xyz="0 0 0"
-        rpy="0 0 0" />
-      <geometry>
-        <mesh
-          filename="file://$(find cra_description)/meshes/cr20/Link3.STL" />
-      </geometry>
-      <material
-        name="">
-        <color
-          rgba="0.792156862745098 0.819607843137255 0.933333333333333 1" />
-      </material>
-    </visual>
-    <collision>
-      <origin
-        xyz="0 0 0"
-        rpy="0 0 0" />
-      <geometry>
-        <mesh
-          filename="file://$(find cra_description)/meshes/cr20/Link3.STL" />
-      </geometry>
-    </collision>
-  </link>
-  <joint
-    name="joint3"
-    type="revolute">
-    <origin
-      xyz="-0.8252 0 0.0468"
-      rpy="0 0 0" />
-    <parent
-      link="Link2" />
-    <child
-      link="Link3" />
-    <axis
-      xyz="0 0 1" />
-    <limit
-      lower="-2.9"
-      upper="2.9"
-      effort="150"
-      velocity="3.14" />
-  </joint>
-  <link
-    name="Link4">
-    <inertial>
-      <origin
-        xyz="1.09076486456641E-07 -0.0757301256894509 1.20551504334543E-08"
-        rpy="0 0 0" />
-      <mass
-        value="3.0" />
-      <inertia
-        ixx="0.01"
-        ixy="0"
-        ixz="0"
-        iyy="0.01"
-        iyz="0"
-        izz="0.005" />
-    </inertial>
-    <visual>
-      <origin
-        xyz="0 0 0"
-        rpy="0 0 0" />
-      <geometry>
-        <mesh
-          filename="file://$(find cra_description)/meshes/cr20/Link4.STL" />
-      </geometry>
-      <material
-        name="">
-        <color
-          rgba="0.792156862745098 0.819607843137255 0.933333333333333 1" />
-      </material>
-    </visual>
-    <collision>
-      <origin
-        xyz="0 0 0"
-        rpy="0 0 0" />
-      <geometry>
-        <mesh
-          filename="file://$(find cra_description)/meshes/cr20/Link4.STL" />
-      </geometry>
-    </collision>
-  </link>
-  <joint
-    name="joint4"
-    type="revolute">
-    <origin
-      xyz="-0.746 0 0.1288"
-      rpy="0 0 -1.5708" />
-    <parent
-      link="Link3" />
-    <child
-      link="Link4" />
-    <axis
-      xyz="0 0 1" />
-    <limit
-      lower="-6.28"
-      upper="6.28"
-      effort="50"
-      velocity="3.14" />
-  </joint>
-  <link
-    name="Link5">
-    <inertial>
-      <origin
-        xyz="-1.06334234349293E-07 0.075730132822537 4.0368623999143E-09"
-        rpy="0 0 0" />
-      <mass
-        value="2.0" />
-      <inertia
-        ixx="0.005"
-        ixy="0"
-        ixz="0"
-        iyy="0.005"
-        iyz="0"
-        izz="0.003" />
-    </inertial>
-    <visual>
-      <origin
-        xyz="0 0 0"
-        rpy="0 0 0" />
-      <geometry>
-        <mesh
-          filename="file://$(find cra_description)/meshes/cr20/Link5.STL" />
-      </geometry>
-      <material
-        name="">
-        <color
-          rgba="0.792156862745098 0.819607843137255 0.933333333333333 1" />
-      </material>
-    </visual>
-    <collision>
-      <origin
-        xyz="0 0 0"
-        rpy="0 0 0" />
-      <geometry>
-        <mesh
-          filename="file://$(find cra_description)/meshes/cr20/Link5.STL" />
-      </geometry>
-    </collision>
-  </link>
-  <joint
-    name="joint5"
-    type="revolute">
-    <origin
-      xyz="0 -0.1288 0"
-      rpy="1.5708 0 0" />
-    <parent
-      link="Link4" />
-    <child
-      link="Link5" />
-    <axis
-      xyz="0 0 1" />
-    <limit
-      lower="-6.28"
-      upper="6.28"
-      effort="50"
-      velocity="3.14" />
-  </joint>
-  <link
-    name="Link6">
-    <inertial>
-      <origin
-        xyz="0.0154576401891996 0.658802608062882 -0.213462466800391"
-        rpy="0 0 0" />
-      <mass
-        value="1.0" />
-      <inertia
-        ixx="0.002"
-        ixy="0"
-        ixz="0"
-        iyy="0.002"
-        iyz="0"
-        izz="0.001" />
-    </inertial>
-    <visual>
-      <origin
-        xyz="0 0 0"
-        rpy="0 0 0" />
-      <geometry>
-        <mesh
-          filename="file://$(find cra_description)/meshes/cr20/Link6.STL" />
-      </geometry>
-      <material
-        name="">
-        <color
-          rgba="0.792156862745098 0.819607843137255 0.933333333333333 1" />
-      </material>
-    </visual>
-    <collision>
-      <origin
-        xyz="0 0 0"
-        rpy="0 0 0" />
-      <geometry>
-        <mesh
-          filename="file://$(find cra_description)/meshes/cr20/Link6.STL" />
-      </geometry>
-    </collision>
-  </link>
-  <joint
-    name="joint6"
-    type="revolute">
-    <origin
-      xyz="0 0.1365 0"
-      rpy="-1.5708 0 0" />
-    <parent
-      link="Link5" />
-    <child
-      link="Link6" />
-    <axis
-      xyz="0 0 1" />
-    <limit
-      lower="-6.28"
-      upper="6.28"
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
File: install/cra_description/share/cra_description/urdf/d435i_with_gazebo.urdf.xacro (robot description, xacro)
@@ -1,72 +1 @@
-<?xml version="1.0"?>
-<robot xmlns:xacro="http://www.ros.org/wiki/xacro">
-  <!-- Include the OFFICIAL Intel RealSense D435i model -->
-  <xacro:include filename="$(find realsense2_description)/urdf/_d435i.urdf.xacro"/>
-  <xacro:macro name="d435i_with_gazebo" params="parent *origin name:=camera use_nominal_extrinsics:=false">
-    <!-- Use official model for geometry, kinematics, and visuals -->
-    <xacro:sensor_d435i
-      parent="${parent}"
-      name="${name}"
-      use_nominal_extrinsics="${use_nominal_extrinsics}">
-      <xacro:insert_block name="origin"/>
-    </xacro:sensor_d435i>
-    <!-- Gazebo RGB Camera Sensor -->
-    <gazebo reference="${name}_bottom_screw_frame">
-      <sensor name="${name}_color_sensor" type="camera">
-        <pose>0.0106 0.0325 0.0125 0 0 0</pose>
-        <always_on>1</always_on>
-        <update_rate>30</update_rate>
-        <visualize>true</visualize>
-        <topic>${name}/camera/color/image_raw</topic>
-        <enable_metrics>false</enable_metrics>
-        <camera>
-          <horizontal_fov>1.211</horizontal_fov>
-          <image>
-            <width>1920</width>
-            <height>1080</height>
-            <format>RGB_INT8</format>
-          </image>
-          <clip>
-            <near>0.1</near>
-            <far>100</far>
-          </clip>
-          <noise>
-            <type>gaussian</type>
-            <mean>0.0</mean>
-            <stddev>0.007</stddev>
-          </noise>
-        </camera>
-        <ignition_frame_id>${name}_color_optical_frame</ignition_frame_id>
-      </sensor>
-    </gazebo>
-    <!-- Gazebo Depth Camera Sensor -->
-    <gazebo reference="${name}_bottom_screw_frame">
-      <sensor name="${name}_depth_sensor" type="depth_camera">
-        <pose>0.0106 0.0175 0.0125 0 0 0</pose>
-        <always_on>1</always_on>
-        <update_rate>30</update_rate>
-        <visualize>true</visualize>
-        <topic>${name}/camera/depth</topic>
-        <enable_metrics>false</enable_metrics>
-        <camera>
-          <horizontal_fov>1.211</horizontal_fov>
-          <image>
-            <width>1280</width>
-            <height>720</height>
-            <format>R_FLOAT32</format>
-          </image>
-          <clip>
-            <near>0.1</near>
-            <far>10.0</far>
-          </clip>
-          <noise>
-            <type>gaussian</type>
-            <mean>0.0</mean>
-            <stddev>0.01</stddev>
-          </noise>
-        </camera>
-        <ignition_frame_id>${name}_depth_optical_frame</ignition_frame_id>
-      </sensor>
-    </gazebo>
-  </xacro:macro>
-</robot>
+/home/iudc/dobot_ws/src/DOBOT_6Axis_ROS2_V4/cra_description/urdf/d435i_with_gazebo.urdf.xacro
